Commit message: added camera, no depth yet

File: src/tars4_1_urdf/urdf/tars4.urdf.xacro (robot description, xacro)
@@ -281,4 +281,52 @@
       velocity="1.5" />
   </joint>
+  <joint name="camera_joint" type="fixed">
+        <parent link="base_link"/>
+        <child link="camera_link"/>
+        <origin xyz="0.32636 0 0.65905" rpy="0 0 0"/>
+    </joint>
+    <link name="camera_link">
+        <visual>
+            <geometry>
+                <box size="0.033 0.175 0.03"/>
+                <material
+                name="">
+                <color
+                rgba="0 0 0 1" />
+               </material>
+            </geometry>
+        </visual>
+    </link>
+    <joint name="camera_optical_joint" type="fixed">
+        <parent link="camera_link"/>
+        <child link="camera_link_optical"/>
+        <origin xyz="0 0 0" rpy="-1.57079632679 0 -1.57079632679"/>
+    </joint>
+    <link name="camera_link_optical"></link>
+    <gazebo reference="camera_link">
+        <material>Gazebo/Red</material>
+        <sensor name="camera" type="depth">
+            <pose> 0 0 0 0 0 0 </pose>
+            <visualize>true</visualize>
+            <update_rate>30</update_rate>
+            <camera>
+                <horizontal_fov>1.57079632679</horizontal_fov>
+                <image>
+                    <format>B8G8R8</format>
+                    <width>1920</width>
+                    <height>1080</height>
+                </image>
+                <clip>
+                    <near>0.5</near>
+                    <far>25.0</far>
+                </clip>
+            </camera>
+            <plugin name="camera_controller" filename="libgazebo_ros_camera.so">
+                <frame_name>camera_link_optical</frame_name>
+                <min_depth>0.5</min_depth>
+                <max_depth>25</max_depth>
+            </plugin>
+        </sensor>
+    </gazebo>
 <gazebo>
   <plugin name="skid_steer_drive_controller" filename="libgazebo_ros_skid_steer_drive.so">

Commit message: added R_L Stereo Cam

File: src/tars4_1_urdf/urdf/tars4.urdf.xacro (robot description, xacro)
@@ -281,10 +281,11 @@
       velocity="1.5" />
   </joint>
-  <joint name="camera_joint" type="fixed">
+<!--right camera ..............................................-->
+  <joint name="r_camera_joint" type="fixed">
         <parent link="base_link"/>
-        <child link="camera_link"/>
-        <origin xyz="0.32636 0 0.65905" rpy="0 0 0"/>
+        <child link="r_camera_link"/>
+        <origin xyz="0.32636 0.06 0.65905" rpy="0 0 0"/>
     </joint>
-    <link name="camera_link">
+    <link name="r_camera_link">
         <visual>
             <geometry>
@@ -298,13 +299,13 @@
         </visual>
     </link>
-    <joint name="camera_optical_joint" type="fixed">
-        <parent link="camera_link"/>
-        <child link="camera_link_optical"/>
+    <joint name="r_camera_optical_joint" type="fixed">
+        <parent link="r_camera_link"/>
+        <child link="r_camera_link_optical"/>
         <origin xyz="0 0 0" rpy="-1.57079632679 0 -1.57079632679"/>
     </joint>
-    <link name="camera_link_optical"></link>
-    <gazebo reference="camera_link">
+    <link name="r_camera_link_optical"></link>
+    <gazebo reference="r_camera_link">
         <material>Gazebo/Red</material>
-        <sensor name="camera" type="depth">
+        <sensor name="camera" type="camera">
             <pose> 0 0 0 0 0 0 </pose>
             <visualize>true</visualize>
@@ -323,5 +324,7 @@
             </camera>
             <plugin name="camera_controller" filename="libgazebo_ros_camera.so">
-                <frame_name>camera_link_optical</frame_name>
+                <frame_name>r_camera_link_optical</frame_name>
+                <cameraName>r_camera</cameraName>
+                <imageTopicName>r_camera/r_image_raw</imageTopicName>
                 <min_depth>0.5</min_depth>
                 <max_depth>25</max_depth>
@@ -329,5 +332,58 @@
         </sensor>
     </gazebo>
-<gazebo>
+<!-- left camera .............................................. -->
+  <joint name="l_camera_joint" type="fixed">
+        <parent link="base_link"/>
+        <child link="l_camera_link"/>
+        <origin xyz="0.32636 -0.06 0.65905" rpy="0 0 0"/>
+    </joint>
+    <link name="l_camera_link">
+        <visual>
+            <geometry>
+                <box size="0.033 0.175 0.03"/>
+                <material
+                name="">
+                <color
+                rgba="0 0 0 1" />
+               </material>
+            </geometry>
+        </visual>
+    </link>
+    <joint name="l_camera_optical_joint" type="fixed">
+        <parent link="l_camera_link"/>
+        <child link="l_camera_link_optical"/>
+        <origin xyz="0 0 0" rpy="-1.57079632679 0 -1.57079632679"/>
+    </joint>
+    <link name="l_camera_link_optical"></link>
+    <gazebo reference="l_camera_link">
+        <material>Gazebo/Red</material>
+        <sensor name="l_camera" type="camera">
+            <pose> 0 0 0 0 0 0 </pose>
+            <visualize>true</visualize>
+            <update_rate>30</update_rate>
+            <camera>
+                <horizontal_fov>1.57079632679</horizontal_fov>
+                <image>
+                    <format>B8G8R8</format>
+                    <width>1920</width>
+                    <height>1080</height>
+                </image>
+                <clip>
+                    <near>0.5</near>
+                    <far>25.0</far>
+                </clip>
+            </camera>
+            <plugin name="camera_controller" filename="libgazebo_ros_camera.so">
+                <cameraName>l_camera</cameraName>
+                <frame_name>l_camera_link_optical</frame_name>
+                <imageTopicName>l_camera/l_image_raw</imageTopicName>
+                <cameraInfoTopicName>l_camera/l_camera_info</cameraInfoTopicName>
+                <min_depth>0.5</min_depth>
+                <max_depth>25</max_depth>
+            </plugin>
+        </sensor>
+    </gazebo>
+ <!--Skid Steer Plugin ..............................................-->
+ <gazebo>
   <plugin name="skid_steer_drive_controller" filename="libgazebo_ros_skid_steer_drive.so">
     <updateRate>100.0</updateRate>

Commit message: added kinect depth camera

File: src/tars4_1_urdf/urdf/tars4.urdf.xacro (robot description, xacro)
@@ -9,5 +9,5 @@
     <inertial>
       <origin
-        xyz="0.0732745727557489 0.000493510970256962 0.413214837428418"
+        xyz="0 0 0"
         rpy="0 0 0" />
       <mass
@@ -285,5 +285,5 @@
         <parent link="base_link"/>
         <child link="r_camera_link"/>
-        <origin xyz="0.32636 0.06 0.65905" rpy="0 0 0"/>
+        <origin xyz="0.32636 0 0.65905" rpy="0 0 0"/>
     </joint>
     <link name="r_camera_link">
@@ -307,6 +307,6 @@
     <gazebo reference="r_camera_link">
         <material>Gazebo/Red</material>
-        <sensor name="camera" type="camera">
-            <pose> 0 0 0 0 0 0 </pose>
+        <sensor name="camera" type="depth">
+            <pose> 0 0 0 0 -1.57079632679 0 </pose>
             <visualize>true</visualize>
             <update_rate>30</update_rate>
@@ -314,5 +314,5 @@
                 <horizontal_fov>1.57079632679</horizontal_fov>
                 <image>
-                    <format>B8G8R8</format>
+                    <format>R8G8B8</format>
                     <width>1920</width>
                     <height>1080</height>
@@ -323,17 +323,36 @@
                 </clip>
             </camera>
-            <plugin name="camera_controller" filename="libgazebo_ros_camera.so">
-                <cameraName>r_camera</cameraName>
-                <frame_name>r_camera_link_optical</frame_name>
-                <imageTopicName>/stereo/right/image_raw</imageTopicName>
-                <cameraInfoTopicName>/stereo/right/camera_info</cameraInfoTopicName>
-                <broadcastTF>true</broadcastTF>
-                <min_depth>0.5</min_depth>
-                <max_depth>25</max_depth>
+            <plugin name="camera_controller" filename="libDepthCameraPlugin.so">
+            <CxPrime>0</CxPrime>
+            <updateRate>10.0</updateRate>
+            <cameraName>depth_cam1</cameraName>
+            <frameName>r_camera_link_optical</frameName>
+            <hackBaseline>0.07</hackBaseline>
+            <distortionK1>1.0</distortionK1>
+            <distortionK2>1.0</distortionK2>
+            <distortionK3>1.0</distortionK3>
+            <distortionT1>1.0</distortionT1>
+            <distortionT2>1.0</distortionT2>
+          </plugin>
+          <plugin name="kinect" filename="libgazebo_ros_openni_kinect.so">
+              <CxPrime>0</CxPrime>
+              <updateRate>10.0</updateRate>
+              <imageTopicName>image_raw</imageTopicName>
+              <pointCloudTopicName>points</pointCloudTopicName>
+              <depthImageTopicName>image_depth</depthImageTopicName>
+              <depthImageCameraInfoTopicName>depth_camera_info</depthImageCameraInfoTopicName>
+              <pointCloudCutoff>0.001</pointCloudCutoff>
+              <cameraName>kinect</cameraName>
+              <frameName>r_camera_link_optical</frameName>
+              <distortionK1>0.00000001</distortionK1>
+              <distortionK2>0.00000001</distortionK2>
+              <distortionK3>0.00000001</distortionK3>
+              <distortionT1>0.00000001</distortionT1>
+              <distortionT2>0.00000001</distortionT2>
             </plugin>
         </sensor>
     </gazebo>
 <!-- left camera .............................................. -->
-  <joint name="l_camera_joint" type="fixed">
+  <!-- <joint name="l_camera_joint" type="fixed">
         <parent link="base_link"/>
         <child link="l_camera_link"/>
@@ -363,9 +382,9 @@
             <pose> 0 0 0 0 0 0 </pose>
             <visualize>true</visualize>
-            <update_rate>30</update_rate>
+            <update_rate>10</update_rate>
             <camera>
                 <horizontal_fov>1.57079632679</horizontal_fov>
                 <image>
-                    <format>B8G8R8</format>
+                    <format>R8G8B8</format>
                     <width>1920</width>
                     <height>1080</height>
@@ -381,4 +400,5 @@
                 <imageTopicName>/stereo/left/image_raw</imageTopicName>
                 <cameraInfoTopicName>/stereo/left/camera_info</cameraInfoTopicName>
+                <frame_name>1_laser_frame</frame_name>
                 <broadcastTF>true</broadcastTF>
                 <min_depth>0.5</min_depth>
@@ -386,5 +406,5 @@
             </plugin>
         </sensor>
-    </gazebo>
+    </gazebo> -->
  <!--Skid Steer Plugin ..............................................-->
  <gazebo>

Commit message: updated to match zed 1 params

File: src/tars4_1_urdf/urdf/tars4.urdf.xacro (robot description, xacro)
@@ -282,10 +282,10 @@
   </joint>
 <!--right camera ..............................................-->
-  <joint name="r_camera_joint" type="fixed">
+  <!-- <joint name="depth_camera_joint" type="fixed">
         <parent link="base_link"/>
-        <child link="r_camera_link"/>
+        <child link="depth_camera_link"/>
         <origin xyz="0.32636 0 0.65905" rpy="0 0 0"/>
     </joint>
-    <link name="r_camera_link">
+    <link name="depth_camera_link">
         <visual>
             <geometry>
@@ -299,11 +299,69 @@
         </visual>
     </link>
-    <joint name="r_camera_optical_joint" type="fixed">
-        <parent link="r_camera_link"/>
-        <child link="r_camera_link_optical"/>
+    <joint name="depth_camera_optical_joint" type="fixed">
+        <parent link="depth_camera_link"/>
+        <child link="depth_camera_link_optical"/>
         <origin xyz="0 0 0" rpy="-1.57079632679 0 -1.57079632679"/>
     </joint>
-    <link name="r_camera_link_optical"></link>
-    <gazebo reference="r_camera_link">
+    <link name="depth_camera_link_optical"></link>
+    <gazebo reference="depth_camera_link">
+        <material>Gazebo/Red</material>
+        <sensor name="depth_camera" type="camera">
+            <pose> 0 0 0 0 0 0 </pose>
+            <visualize>true</visualize>
+            <update_rate>10</update_rate>
+            <camera>
+                <horizontal_fov>1.57079632679</horizontal_fov>
+                <image>
+                    <format>R8G8B8</format>
+                    <width>1920</width>
+                    <height>1080</height>
+                </image>
+                <clip>
+                    <near>0.5</near>
+                    <far>25.0</far>
+                </clip>
+            </camera>
+            <plugin name="camera_controller" filename="libgazebo_ros_camera.so">
+                <cameraName>depth_camera</cameraName>
+                <frame_name>depth_camera_link_optical</frame_name>
+                <imageTopicName>/stereo/right/image_raw</imageTopicName>
+                <cameraInfoTopicName>/stereo/right/camera_info</cameraInfoTopicName>
+                <broadcastTF>true</broadcastTF>
+                <hackBaseline>0.07</hackBaseline>
+                <distortionK1>0.0</distortionK1>
+                <distortionK2>0.0</distortionK2>
+                <distortionK3>0.0</distortionK3>
+                <distortionT1>0.0</distortionT1>
+                <distortionT2>0.0</distortionT2>
+                <min_depth>0.5</min_depth>
+                <max_depth>25</max_depth>
+            </plugin>
+        </sensor>
+    </gazebo> -->
+  <joint name="depth_camera_joint" type="fixed">
+        <parent link="base_link"/>
+        <child link="depth_camera_link"/>
+        <origin xyz="0.32636 0 0.65905" rpy="0 0 0"/>
+    </joint>
+    <link name="depth_camera_link">
+        <visual>
+            <geometry>
+                <box size="0.033 0.175 0.03"/>
+                <material
+                name="">
+                <color
+                rgba="0 0 0 1" />
+               </material>
+            </geometry>
+        </visual>
+    </link>
+    <joint name="depth_camera_optical_joint" type="fixed">
+        <parent link="depth_camera_link"/>
+        <child link="depth_camera_link_optical"/>
+        <origin xyz="0 0 0" rpy="-1.57079632679 0 -1.57079632679"/>
+    </joint>
+    <link name="depth_camera_link_optical"></link>
+    <gazebo reference="depth_camera_link">
         <material>Gazebo/Red</material>
         <sensor name="camera" type="depth">
@@ -325,8 +383,8 @@
             <plugin name="camera_controller" filename="libDepthCameraPlugin.so">
             <CxPrime>0</CxPrime>
-            <updateRate>10.0</updateRate>
+            <updateRate>30.0</updateRate>
             <cameraName>depth_cam1</cameraName>
-            <frameName>r_camera_link_optical</frameName>
-            <hackBaseline>0.07</hackBaseline>
+            <frameName>depth_camera_link_optical</frameName>
+            <hackBaseline>0.012</hackBaseline>
             <distortionK1>1.0</distortionK1>
             <distortionK2>1.0</distortionK2>
@@ -337,5 +395,5 @@
           <plugin name="kinect" filename="libgazebo_ros_openni_kinect.so">
               <CxPrime>0</CxPrime>
-              <updateRate>10.0</updateRate>
+              <updateRate>30.0</updateRate>
               <imageTopicName>image_raw</imageTopicName>
               <pointCloudTopicName>points</pointCloudTopicName>
@@ -344,5 +402,5 @@
               <pointCloudCutoff>0.001</pointCloudCutoff>
               <cameraName>kinect</cameraName>
-              <frameName>r_camera_link_optical</frameName>
+              <frameName>depth_camera_link_optical</frameName>
               <distortionK1>0.00000001</distortionK1>
               <distortionK2>0.00000001</distortionK2>
@@ -357,5 +415,5 @@
         <parent link="base_link"/>
         <child link="l_camera_link"/>
-        <origin xyz="0.32636 -0.06 0.65905" rpy="0 0 0"/>
+        <origin xyz="0.32636 0 0.65905" rpy="0 0 0"/>
     </joint>
     <link name="l_camera_link">
@@ -396,10 +454,16 @@
             </camera>
             <plugin name="camera_controller" filename="libgazebo_ros_camera.so">
+              <alwaysOn>true</alwaysOn>
                 <cameraName>l_camera</cameraName>
                 <frame_name>l_camera_link_optical</frame_name>
                 <imageTopicName>/stereo/left/image_raw</imageTopicName>
                 <cameraInfoTopicName>/stereo/left/camera_info</cameraInfoTopicName>
-                <frame_name>1_laser_frame</frame_name>
                 <broadcastTF>true</broadcastTF>
+                <hackBaseline>0.07</hackBaseline>
+                <distortionK1>0.0</distortionK1>
+                <distortionK2>0.0</distortionK2>
+                <distortionK3>0.0</distortionK3>
+                <distortionT1>0.0</distortionT1>
+                <distortionT2>0.0</distortionT2>
                 <min_depth>0.5</min_depth>
                 <max_depth>25</max_depth>
@@ -409,5 +473,5 @@
  <!--Skid Steer Plugin ..............................................-->
  <gazebo>
-  <plugin name="skid_steer_drive_controller" filename="libgazebo_ros_skid_steer_drive.so">
+  <plugin name="skid_steedepth_drive_controller" filename="libgazebo_ros_skid_steedepth_drive.so">
     <updateRate>100.0</updateRate>
     <robotNamespace>/</robotNamespace>

Commit message: need to add ultrasonic or lidar

File: src/tars4_1_urdf/urdf/tars4.urdf.xacro (robot description, xacro)
@@ -281,63 +281,5 @@
       velocity="1.5" />
   </joint>
-<!--right camera ..............................................-->
-  <!-- <joint name="depth_camera_joint" type="fixed">
-        <parent link="base_link"/>
-        <child link="depth_camera_link"/>
-        <origin xyz="0.32636 0 0.65905" rpy="0 0 0"/>
-    </joint>
-    <link name="depth_camera_link">
-        <visual>
-            <geometry>
-                <box size="0.033 0.175 0.03"/>
-                <material
-                name="">
-                <color
-                rgba="0 0 0 1" />
-               </material>
-            </geometry>
-        </visual>
-    </link>
-    <joint name="depth_camera_optical_joint" type="fixed">
-        <parent link="depth_camera_link"/>
-        <child link="depth_camera_link_optical"/>
-        <origin xyz="0 0 0" rpy="-1.57079632679 0 -1.57079632679"/>
-    </joint>
-    <link name="depth_camera_link_optical"></link>
-    <gazebo reference="depth_camera_link">
-        <material>Gazebo/Red</material>
-        <sensor name="depth_camera" type="camera">
-            <pose> 0 0 0 0 0 0 </pose>
-            <visualize>true</visualize>
-            <update_rate>10</update_rate>
-            <camera>
-                <horizontal_fov>1.57079632679</horizontal_fov>
-                <image>
-                    <format>R8G8B8</format>
-                    <width>1920</width>
-                    <height>1080</height>
-                </image>
-                <clip>
-                    <near>0.5</near>
-                    <far>25.0</far>
-                </clip>
-            </camera>
-            <plugin name="camera_controller" filename="libgazebo_ros_camera.so">
-                <cameraName>depth_camera</cameraName>
-                <frame_name>depth_camera_link_optical</frame_name>
-                <imageTopicName>/stereo/right/image_raw</imageTopicName>
-                <cameraInfoTopicName>/stereo/right/camera_info</cameraInfoTopicName>
-                <broadcastTF>true</broadcastTF>
-                <hackBaseline>0.07</hackBaseline>
-                <distortionK1>0.0</distortionK1>
-                <distortionK2>0.0</distortionK2>
-                <distortionK3>0.0</distortionK3>
-                <distortionT1>0.0</distortionT1>
-                <distortionT2>0.0</distortionT2>
-                <min_depth>0.5</min_depth>
-                <max_depth>25</max_depth>
-            </plugin>
-        </sensor>
-    </gazebo> -->
+ <!-- Depth camera plugin ..................................................................................-->
   <joint name="depth_camera_joint" type="fixed">
         <parent link="base_link"/>
@@ -411,64 +353,4 @@
         </sensor>
     </gazebo>
-<!-- left camera .............................................. -->
-  <!-- <joint name="l_camera_joint" type="fixed">
-        <parent link="base_link"/>
-        <child link="l_camera_link"/>
-        <origin xyz="0.32636 0 0.65905" rpy="0 0 0"/>
-    </joint>
-    <link name="l_camera_link">
-        <visual>
-            <geometry>
-                <box size="0.033 0.175 0.03"/>
-                <material
-                name="">
-                <color
-                rgba="0 0 0 1" />
-               </material>
-            </geometry>
-        </visual>
-    </link>
-    <joint name="l_camera_optical_joint" type="fixed">
-        <parent link="l_camera_link"/>
-        <child link="l_camera_link_optical"/>
-        <origin xyz="0 0 0" rpy="-1.57079632679 0 -1.57079632679"/>
-    </joint>
-    <link name="l_camera_link_optical"></link>
-    <gazebo reference="l_camera_link">
-        <material>Gazebo/Red</material>
-        <sensor name="l_camera" type="camera">
-            <pose> 0 0 0 0 0 0 </pose>
-            <visualize>true</visualize>
-            <update_rate>10</update_rate>
-            <camera>
-                <horizontal_fov>1.57079632679</horizontal_fov>
-                <image>
-                    <format>R8G8B8</format>
-                    <width>1920</width>
-                    <height>1080</height>
-                </image>
-                <clip>
-                    <near>0.5</near>
-                    <far>25.0</far>
-                </clip>
-            </camera>
-            <plugin name="camera_controller" filename="libgazebo_ros_camera.so">
-              <alwaysOn>true</alwaysOn>
-                <cameraName>l_camera</cameraName>
-                <frame_name>l_camera_link_optical</frame_name>
-                <imageTopicName>/stereo/left/image_raw</imageTopicName>
-                <cameraInfoTopicName>/stereo/left/camera_info</cameraInfoTopicName>
-                <broadcastTF>true</broadcastTF>
-                <hackBaseline>0.07</hackBaseline>
-                <distortionK1>0.0</distortionK1>
-                <distortionK2>0.0</distortionK2>
-                <distortionK3>0.0</distortionK3>
-                <distortionT1>0.0</distortionT1>
-                <distortionT2>0.0</distortionT2>
-                <min_depth>0.5</min_depth>
-                <max_depth>25</max_depth>
-            </plugin>
-        </sensor>
-    </gazebo> -->
  <!--Skid Steer Plugin ..............................................-->
  <gazebo>
