Commit message: added front ir sensor

File: src/tars4_1_urdf/urdf/tars4.urdf.xacro (robot description, xacro)
@@ -12,5 +12,5 @@
         rpy="0 0 0" />
       <mass
-        value="26.298368938694" />
+        value="50" />
       <inertia
         ixx="1.2118547835405"
@@ -375,3 +375,66 @@
   </plugin>
 </gazebo>
+<!--IR/SONAR Plugin ..............................................-->
+<joint name="ir_front_joint" type="fixed">
+    <axis xyz="0 1 0" />
+    <origin rpy="0 0 0" xyz="0.5 0 0" />
+    <parent link="base_link"/>
+    <child link="base_ir_front"/>
+</joint>
+<link name="base_ir_front">
+    <collision>
+      <origin xyz="0 0 0" rpy="0 0 0"/>
+      <geometry>
+        <box size="0.01 0.01 0.01"/>
+      </geometry>
+    </collision>
+    <visual>
+      <origin xyz="0 0 0" rpy="0 0 0"/>
+      <geometry>
+        <box size="0.01 0.01 0.01"/>
+      </geometry>
+    </visual>
+    <inertial>
+      <mass value="1e-5" />
+      <origin xyz="0 0 0" rpy="0 0 0"/>
+      <inertia ixx="1e-6" ixy="0" ixz="0" iyy="1e-6" iyz="0"      izz="1e-6" />
+    </inertial>
+</link>
+ <gazebo reference="base_ir_front">
+   <sensor type="ray" name="TeraRanger">
+      <pose>0 0 0 0 0 0</pose>
+      <visualize>true</visualize>
+      <update_rate>50</update_rate>
+      <ray>
+         <scan>
+            <horizontal>
+               <samples>10</samples>
+               <resolution>1</resolution>
+               <min_angle>-0.654498</min_angle>
+               <max_angle>0.654498</max_angle>
+            </horizontal>
+            <vertical>
+               <samples>10</samples>
+               <resolution>1</resolution>
+               <min_angle>-0.654498</min_angle>
+               <max_angle>0.654498</max_angle>
+            </vertical>
+         </scan>
+         <range>
+            <min>0.2</min>
+            <max>8</max>
+            <resolution>0.02</resolution>
+         </range>
+      </ray>
+      <plugin filename="libgazebo_ros_range.so" name="gazebo_ros_range">
+         <gaussianNoise>0.005</gaussianNoise>
+         <alwaysOn>true</alwaysOn>
+         <updateRate>50</updateRate>
+         <topicName>sensor/ir_front</topicName>
+         <frameName>base_ir_front</frameName>
+         <radiation>INFRARED</radiation>
+         <fov>1.309</fov>
+      </plugin>
+   </sensor>
+   </gazebo>
 </robot>
