Commit message: added weighted TARS5

File: src/TARS5_URDF/urdf/TARS5_URDF.urdf (robot description, URDF)
Before this commit: robot TARS5_URDF, 6 links, 5 joints
Links:
- link base_link: mass 36.0649927126506 -> 95

Commit message: added new TARS campus world, segment code

File: src/TARS5_URDF/urdf/TARS5_URDF.urdf (robot description, URDF)
Before this commit: robot TARS5_URDF, 6 links, 5 joints
Links:
- added link depth_camera_link; visual box size=0.033 0.175 0.03
- added link depth_camera_link_optical
Joints:
- added joint depth_camera_joint: type fixed, parent base_link, child depth_camera_link, origin xyz=0.32636 0 0.65905 rpy=0 0 0
- added joint depth_camera_optical_joint: type fixed, parent depth_camera_link, child depth_camera_link_optical, origin xyz=0 0 0 rpy=-1.57079632679 0 -1.57079632679

Commit message: added segmentation model

File: src/TARS5_URDF/urdf/TARS5_URDF.urdf (robot description, URDF)
Before this commit: robot TARS5_URDF, 8 links, 7 joints
Links:
- removed link base_ir_front
Joints:
- removed joint ir_front_joint
